Commit message: fixup indention

File: osrf_gear/launch/ur10/vacuum_gripper.urdf.xacro (robot description, xacro)
@@ -5,8 +5,8 @@
     <inertial>
       <origin xyz="0 0 0" rpy="0 0 0" />
-        <inertia ixx="0.0000063" ixy="0" ixz="0"
-                 iyy="0.0000063" iyz="0"
-                 izz="0.000025" />
-        <mass value="0.01" />
+      <inertia ixx="0.0000063" ixy="0" ixz="0"
+               iyy="0.0000063" iyz="0"
+               izz="0.000025" />
+      <mass value="0.01" />
     </inertial>
     <visual>
