Commit message: working test of the vacuum gripper

File: osrf_gear/launch/ur10/ur10_with_vacuum_gripper.urdf.xacro (robot description, xacro)
@@ -10,7 +10,9 @@
   <!-- vacuum gripper -->
   <xacro:include filename="$(find osrf_gear)/launch/ur10/vacuum_gripper.urdf.xacro" />
-  <xacro:create_vacuum_gripper />
-  <joint name="vacuum_gripper_joint" type="fixed">
+  <xacro:create_vacuum_gripper suction_cup_link_name="robot::vacuum_gripper_link" />
+  <joint name="vacuum_gripper_joint" type="revolute">
     <origin xyz="0 0.1 0" rpy="${90 * 0.0174533} 0 0" />
+    <axis xyz="0 0 1" />
+    <limit lower="0" upper="0" effort="0" velocity="0" />
     <parent link="wrist_3_link" />
     <child link="vacuum_gripper_link" />

File: osrf_gear/launch/ur10/vacuum_gripper.urdf.xacro (robot description, xacro)
@@ -1,5 +1,5 @@
 <?xml version="1.0"?>
 <robot xmlns:xacro="http://www.ros.org/wiki/xacro">
-<xacro:macro name="create_vacuum_gripper">
+<xacro:macro name="create_vacuum_gripper" params="suction_cup_link_name">
   <link name="vacuum_gripper_link">
     <inertial>
@@ -15,6 +15,6 @@
         <cylinder radius="0.05" length="0.01" />
       </geometry>
-      <material name="Black">
-        <color rgba="1.0 1.0 1.0 1.0"/>
+      <material name="SomeColor">
+        <color rgba="1.0 0.0 0.0 1.0"/>
       </material>
     </visual>
@@ -26,4 +26,7 @@
     </collision>
   </link>
+  <gazebo reference="vacuum_gripper_link">
+    <material>Gazebo/Black</material>
+  </gazebo>
   <gazebo>
     <plugin name="ros_vacuum_gripper" filename="libROSVacuumGripperPlugin.so">
@@ -33,5 +36,5 @@
         <min_contact_count>1</min_contact_count>
       </grasp_check>
-      <suction_cup_link>vacuum_gripper_link</suction_cup_link>
+      <suction_cup_link>${suction_cup_link_name}</suction_cup_link>
       <!-- ROS -->
       <robot_namespace>vacuum_gripper</robot_namespace>

Commit message: add linear actuator for arm

File: osrf_gear/launch/ur10/ur10_with_vacuum_gripper.urdf.xacro (robot description, xacro)
@@ -7,5 +7,5 @@
   <xacro:include filename="$(find ur_description)/urdf/ur10.urdf.xacro" />
   <!-- arm -->
-  <xacro:ur10_robot prefix="" joint_limited="false" />
+  <xacro:ur10_robot prefix="" />
   <!-- vacuum gripper -->
   <xacro:include filename="$(find osrf_gear)/launch/ur10/vacuum_gripper.urdf.xacro" />
@@ -19,10 +19,24 @@
     <dynamics damping="0.0" friction="0.0"/>
   </joint>
+  <!-- linear arm actuator -->
+  <xacro:include filename="$(find osrf_gear)/launch/linear_arm_actuator/linear_arm_actuator.urdf.xacro" />
+  <xacro:create_linear_arm_actuator base_link="base_link" />
   <!-- world link -->
   <link name="world" />
   <joint name="world_joint" type="fixed">
     <parent link="world" />
-    <child link="base_link" />
-    <origin xyz="0.0 0.0 0.0" rpy="0.0 0.0 0.0" />
+    <child link="linear_arm_actuator" />
+    <origin xyz="0.0 0.0 0.1" rpy="0.0 0.0 0.0" />
   </joint>
+  <!-- plugin to spawn gazebo scene data into the moveit scene -->
+  <!--
+  <gazebo>
+    <plugin filename="libgazebo_ros_moveit_planning_scene.so" name="gazebo_ros_moveit_planning_scene">
+      <topicName>/planning_scene</topicName>
+      <sceneName>workcell</sceneName>
+      <robotName>robot</robotName>
+      <updatePeriod>0.5</updatePeriod>
+    </plugin>
+  </gazebo>
+  -->
 </robot>

Commit message: Add dumpster to ur10 world

File: osrf_gear/launch/ur10/ur10_with_vacuum_gripper.urdf.xacro (robot description, xacro)
@@ -27,5 +27,5 @@
     <parent link="world" />
     <child link="linear_arm_actuator" />
-    <origin xyz="0.0 0.0 0.1" rpy="0.0 0.0 0.0" />
+    <origin xyz="0.0 0.0 1.0" rpy="0.0 0.0 0.0" />
   </joint>
   <!-- plugin to spawn gazebo scene data into the moveit scene -->

Commit message: remap topics and services for competition to /ariac/*

File: osrf_gear/launch/ur10/ur10_with_vacuum_gripper.urdf.xacro (robot description, xacro)
@@ -27,5 +27,5 @@
     <parent link="world" />
     <child link="linear_arm_actuator" />
-    <origin xyz="0.0 0.0 1.0" rpy="0.0 0.0 0.0" />
+    <origin xyz="0.0 0.0 1.2" rpy="0.0 0.0 0.0" />
   </joint>
   <!-- plugin to spawn gazebo scene data into the moveit scene -->

File: osrf_gear/launch/ur10/vacuum_gripper.urdf.xacro (robot description, xacro)
@@ -38,5 +38,5 @@
       <suction_cup_link>${suction_cup_link_name}</suction_cup_link>
       <!-- ROS -->
-      <robot_namespace>vacuum_gripper</robot_namespace>
+      <robot_namespace>/ariac</robot_namespace>
       <control_topic>vacuum_gripper_control</control_topic>
       <state_topic>vacuum_gripper_state</state_topic>

Commit message: integrate workcell env into ariac.world

File: osrf_gear/launch/ur10/ur10_with_vacuum_gripper.urdf.xacro (robot description, xacro)
@@ -27,5 +27,5 @@
     <parent link="world" />
     <child link="linear_arm_actuator" />
-    <origin xyz="0.0 0.0 1.2" rpy="0.0 0.0 0.0" />
+    <origin xyz="0.0 0.0 1" rpy="0.0 0.0 0.0" />
   </joint>
   <!-- plugin to spawn gazebo scene data into the moveit scene -->

Commit message: reorganize xacro to have urdf entry for each sensor
also fixes the problem where the arm only showed some states

File: osrf_gear/launch/ur10/ur10_with_vacuum_gripper.urdf.xacro (robot description, xacro)
@@ -21,24 +21,3 @@
     <dynamics damping="0.0" friction="0.0"/>
   </joint>
-  <!-- linear arm actuator -->
-  <xacro:include filename="$(find osrf_gear)/launch/linear_arm_actuator/linear_arm_actuator.urdf.xacro" />
-  <xacro:create_linear_arm_actuator base_link="base_link" />
-  <!-- world link -->
-  <link name="world" />
-  <joint name="world_joint" type="fixed">
-    <parent link="world" />
-    <child link="linear_arm_actuator" />
-    <origin xyz="0.0 0.0 1" rpy="0.0 0.0 0.0" />
-  </joint>
-  <!-- plugin to spawn gazebo scene data into the moveit scene -->
-  <!--
-  <gazebo>
-    <plugin filename="libgazebo_ros_moveit_planning_scene.so" name="gazebo_ros_moveit_planning_scene">
-      <topicName>/planning_scene</topicName>
-      <sceneName>workcell</sceneName>
-      <robotName>robot</robotName>
-      <updatePeriod>0.5</updatePeriod>
-    </plugin>
-  </gazebo>
-  -->
 </robot>
