Commit message: Move gripper outside of ur10

File: osrf_gear/launch/ur10/ur10.urdf.xacro (robot description, xacro)
@@ -10,14 +10,3 @@
   <!-- arm -->
   <xacro:ur10_robot prefix="" />
-  <!-- vacuum gripper -->
-  <xacro:include filename="$(find osrf_gear)/launch/ur10/vacuum_gripper.urdf.xacro" />
-  <xacro:create_vacuum_gripper suction_cup_link_name="robot::vacuum_gripper_link" />
-  <joint name="vacuum_gripper_joint" type="revolute">
-    <origin xyz="0 0.1 0" rpy="${90 * 0.0174533} 0 0" />
-    <axis xyz="0 0 1" />
-    <limit lower="0" upper="0" effort="0" velocity="0" />
-    <parent link="wrist_3_link" />
-    <child link="vacuum_gripper_link" />
-    <dynamics damping="0.0" friction="0.0"/>
-  </joint>
 </robot>

File: osrf_gear/launch/vacuum_gripper/vacuum_gripper.urdf.xacro (robot description, xacro)
@@ -1,5 +1,5 @@
 <?xml version="1.0"?>
 <robot xmlns:xacro="http://www.ros.org/wiki/xacro">
-<xacro:macro name="create_vacuum_gripper" params="suction_cup_link_name">
+<xacro:macro name="create_vacuum_gripper" params="wrist_link">
   <link name="vacuum_gripper_link">
     <inertial>
@@ -26,4 +26,12 @@
     </collision>
   </link>
+  <joint name="vacuum_gripper_joint" type="revolute">
+    <origin xyz="0 0.1 0" rpy="${90 * 0.0174533} 0 0" />
+    <axis xyz="0 0 1" />
+    <limit lower="0" upper="0" effort="0" velocity="0" />
+    <parent link="${wrist_link}" />
+    <child link="vacuum_gripper_link" />
+    <dynamics damping="0.0" friction="0.0"/>
+  </joint>
   <gazebo reference="vacuum_gripper_link">
     <material>Gazebo/Black</material>
@@ -36,5 +44,5 @@
         <min_contact_count>1</min_contact_count>
       </grasp_check>
-      <suction_cup_link>${suction_cup_link_name}</suction_cup_link>
+      <suction_cup_link>vacuum_gripper_link</suction_cup_link>
       <!-- ROS -->
       <robot_namespace>/ariac</robot_namespace>
