Commit message: clean up unused files and tune controller more

File: osrf_gear/launch/linear_arm_actuator/linear_arm_actuator.urdf.xacro (robot description, xacro)
@@ -2,5 +2,5 @@
 <robot xmlns:xacro="http://www.ros.org/wiki/xacro">
 <xacro:property name="base_len" value="0.2" />
-<xacro:property name="actuator_len" value="4" />
+<xacro:property name="actuator_len" value="4.6" />
 <xacro:property name="actuator_height" value="0.1" />
 <xacro:macro name="create_linear_arm_actuator" params="base_link">
@@ -39,7 +39,11 @@
            upper="${(actuator_len / 2) - base_len}"
            effort="1000"
-           velocity="1" />
+           velocity="3" />
     <origin xyz="0 0 ${base_len / 2}" rpy="0 0 0" />
+    <dynamics damping="20.0" friction="0.0"/>
   </joint>
+  <gazebo reference="linear_arm_actuator_joint">
+    <implicitSpringDamper>1</implicitSpringDamper>
+  </gazebo>
   <xacro:linear_arm_actuator_transmission />
 </xacro:macro>

File: osrf_gear/vendor/ur_description/urdf/ur10.urdf.xacro (robot description, xacro)
@@ -86,6 +86,9 @@
         <limit lower="${-pi}" upper="${pi}" effort="330.0" velocity="2.16"/>
       </xacro:if>
-      <dynamics damping="0.0" friction="0.0"/>
-    </joint>
+      <dynamics damping="20.0" friction="0.0"/>
+    </joint>
+    <gazebo reference="${prefix}shoulder_pan_joint">
+      <implicitSpringDamper>1</implicitSpringDamper>
+    </gazebo>
     <link name="${prefix}shoulder_link">
       <visual>
@@ -117,6 +120,9 @@
         <limit lower="${-pi}" upper="${pi}" effort="330.0" velocity="2.16"/>
       </xacro:if>
-      <dynamics damping="0.0" friction="0.0"/>
-    </joint>
+      <dynamics damping="20.0" friction="0.0"/>
+    </joint>
+    <gazebo reference="${prefix}shoulder_lift_joint">
+      <implicitSpringDamper>1</implicitSpringDamper>
+    </gazebo>
     <link name="${prefix}upper_arm_link">
       <visual>
@@ -148,6 +154,9 @@
         <limit lower="${-pi}" upper="${pi}" effort="150.0" velocity="3.15"/>
       </xacro:if>
-      <dynamics damping="0.0" friction="0.0"/>
-    </joint>
+      <dynamics damping="20.0" friction="0.0"/>
+    </joint>
+    <gazebo reference="${prefix}elbow_joint">
+      <implicitSpringDamper>1</implicitSpringDamper>
+    </gazebo>
     <link name="${prefix}forearm_link">
       <visual>
@@ -179,6 +188,9 @@
         <limit lower="${-pi}" upper="${pi}" effort="54.0" velocity="3.2"/>
       </xacro:if>
-      <dynamics damping="0.0" friction="0.0"/>
-    </joint>
+      <dynamics damping="1.0" friction="0.0"/>
+    </joint>
+    <gazebo reference="${prefix}wrist_1_joint">
+      <implicitSpringDamper>1</implicitSpringDamper>
+    </gazebo>
     <link name="${prefix}wrist_1_link">
       <visual>
@@ -210,6 +222,9 @@
         <limit lower="${-pi}" upper="${pi}" effort="54.0" velocity="3.2"/>
       </xacro:if>
-      <dynamics damping="0.0" friction="0.0"/>
-    </joint>
+      <dynamics damping="1.0" friction="0.0"/>
+    </joint>
+    <gazebo reference="${prefix}wrist_2_joint">
+      <implicitSpringDamper>1</implicitSpringDamper>
+    </gazebo>
     <link name="${prefix}wrist_2_link">
       <visual>
@@ -241,6 +256,9 @@
         <limit lower="${-pi}" upper="${pi}" effort="54.0" velocity="3.2"/>
       </xacro:if>
-      <dynamics damping="0.0" friction="0.0"/>
-    </joint>
+      <dynamics damping="0.5" friction="0.0"/>
+    </joint>
+    <gazebo reference="${prefix}wrist_3_joint">
+      <implicitSpringDamper>1</implicitSpringDamper>
+    </gazebo>
     <link name="${prefix}wrist_3_link">
       <visual>

Commit message: fine adjustment of physics and controller gains for ur10

File: osrf_gear/launch/linear_arm_actuator/linear_arm_actuator.urdf.xacro (robot description, xacro)
@@ -41,5 +41,5 @@
            velocity="3" />
     <origin xyz="0 0 ${base_len / 2}" rpy="0 0 0" />
-    <dynamics damping="20.0" friction="0.0"/>
+    <dynamics damping="20.0" friction="500.0" />
   </joint>
   <gazebo reference="linear_arm_actuator_joint">

File: osrf_gear/vendor/ur_description/urdf/ur10.urdf.xacro (robot description, xacro)
@@ -81,10 +81,10 @@
       <axis xyz="0 0 1" />
       <xacro:unless value="$(arg joint_limited)">
-        <limit lower="${-2.0 * pi}" upper="${2.0 * pi}" effort="330.0" velocity="2.16"/>
+        <limit lower="${-2.0 * pi}" upper="${2.0 * pi}" effort="${330.0 + 200}" velocity="2.16"/>
       </xacro:unless>
       <xacro:if value="$(arg joint_limited)">
         <limit lower="${-pi}" upper="${pi}" effort="330.0" velocity="2.16"/>
       </xacro:if>
-      <dynamics damping="20.0" friction="0.0"/>
+      <dynamics damping="20.0" friction="20.0"/>
     </joint>
     <gazebo reference="${prefix}shoulder_pan_joint">
