Commit message: Specify drops in yaml config

File: osrf_gear/launch/vacuum_gripper/vacuum_gripper.urdf.xacro (robot description, xacro)
@@ -1,5 +1,5 @@
 <?xml version="1.0"?>
 <robot xmlns:xacro="http://www.ros.org/wiki/xacro">
-<xacro:macro name="create_vacuum_gripper" params="wrist_link">
+<xacro:macro name="create_vacuum_gripper" params="wrist_link *drops">
   <link name="vacuum_gripper_link">
     <inertial>
@@ -44,4 +44,5 @@
         <min_contact_count>1</min_contact_count>
       </grasp_check>
+      <xacro:insert_block name="drops" />
       <suction_cup_link>vacuum_gripper_link</suction_cup_link>
       <!-- ROS -->

Commit message: Only include drops block if necessary

File: osrf_gear/launch/vacuum_gripper/vacuum_gripper.urdf.xacro (robot description, xacro)
@@ -1,5 +1,5 @@
 <?xml version="1.0"?>
 <robot xmlns:xacro="http://www.ros.org/wiki/xacro">
-<xacro:macro name="create_vacuum_gripper" params="wrist_link *drops">
+<xacro:macro name="create_vacuum_gripper" params="wrist_link do_drops *drops">
   <link name="vacuum_gripper_link">
     <inertial>
@@ -44,5 +44,7 @@
         <min_contact_count>1</min_contact_count>
       </grasp_check>
-      <xacro:insert_block name="drops" />
+      <xacro:if value="${do_drops}">
+        <xacro:insert_block name="drops" />
+      </xacro:if>
       <suction_cup_link>vacuum_gripper_link</suction_cup_link>
       <!-- ROS -->

Commit message: Simplify dropped parts xacro

File: osrf_gear/launch/vacuum_gripper/vacuum_gripper.urdf.xacro (robot description, xacro)
@@ -1,5 +1,5 @@
 <?xml version="1.0"?>
 <robot xmlns:xacro="http://www.ros.org/wiki/xacro">
-<xacro:macro name="create_vacuum_gripper" params="wrist_link do_drops *drops">
+<xacro:macro name="create_vacuum_gripper" params="wrist_link **drops_info">
   <link name="vacuum_gripper_link">
     <inertial>
@@ -44,7 +44,5 @@
         <min_contact_count>1</min_contact_count>
       </grasp_check>
-      <xacro:if value="${do_drops}">
-        <xacro:insert_block name="drops" />
-      </xacro:if>
+      <xacro:insert_block name="drops_info" />
       <suction_cup_link>vacuum_gripper_link</suction_cup_link>
       <!-- ROS -->
